File: AXAWIFIESP01.brd (EAGLE design)
At the start: 94 x 27.9 mm, 20 parts, among them IC1 MCP2003, M1 REGMODULE4PIN, M2 ESP01, SW1 RESET, SW2 REFLASH

Commit message: Replace parts using SuperHouse library for 3D models
Parts:
- C2: device freetronics:EIA3216 -> SuperHouse-DiscreteSemi:EIA3216
- C3: device analyzer:UD-6,3X5,8_NICHICON -> SuperHouse-DiscreteSemi:PANASONIC_C
- C4: device freetronics-jon:0603 -> SuperHouse-DiscreteSemi:C0603
- IC1: device freetronics-jon:SOIC8T -> SuperHouse-ICs:SOIC8T
- JP4: device freetronics-master-v1.1:SCREWTERMINAL-3.5MM-2 -> SuperHouse-Connectors:SCREWTERMINAL-3.5MM-2
- LED1: device freetronics-jon:LED-0603 -> SuperHouse-LEDs:LED-0603
- R1, R10, R11, R2, R5, R6, R7, R9: device freetronics-jon:0603 -> SuperHouse-DiscreteSemi:R0603
- SW1, SW2: device freetronics-jon:TACTILE_SWITCH_SMD_2PIN_TINY -> SuperHouse-Switches:TACTILE_SMT_3X4X2
- moved JP4 1.27 mm to (5.08, 5.08)
Routing:
- net DATA: track 71.2 -> 70.4 mm
