File: AXAWIFIESP01.sch (EAGLE design)
At the start: 20 parts, among them IC1 MCP2003, M1 REGMODULE4PIN, M2 ESP01, SW1 RESET, SW2 REFLASH

Commit message: Replace parts using SuperHouse library for 3D models
Parts:
- C2: device freetronics:CAP_POL1206 -> SuperHouse-DiscreteSemi:CAP_POL1206
- C3: device analyzer:CPOL-USUD-6,3X5,8 -> SuperHouse-DiscreteSemi:CAP_POLC
- C4: device freetronics-jon:CAP0603 -> SuperHouse-DiscreteSemi:CAP0603
- IC1: device freetronics-jon:MCP2003 -> SuperHouse-ICs:MCP2003
- JP4: device freetronics-master-v1.1:M023.5MM -> SuperHouse-Connectors:M02-SCREW-3.5MM
- LED1: device freetronics-jon:LED0603 -> SuperHouse-LEDs:LED0603
- R1, R10, R11, R2, R5, R6, R7, R9: device freetronics-jon:RESISTOR0603 -> SuperHouse-DiscreteSemi:RESISTOR0603
- SW1, SW2: device freetronics-jon:TAC_SWITCH_2PIN -> SuperHouse-Switches:TAC_SWITCH_2PINSMT
